File: Homework2/HW2.sch (EAGLE design)
At the start: 21 parts, among them X1 MINI-USB-SCHIELD-32005-301

Commit message: Second Commit
Parts:
- removed J3: (no value), SparkFun-Connectors:CONN_08"
- removed X1: MINI-USB-SCHIELD-32005-301, con-cypressindustries:MINI-USB-SCHIELD-32005-301
- added J4: (no value), SparkFun-Connectors:CONN_08"
- added J6: USB-MB-H, Ilya_Teach:USB-MB-H
- C1, C2, C3, C4: value (none) -> 10uF
- C5: value (none) -> 0.1uF
- R1, R4: value (none) -> 330
- R2, R3: value (none) -> 10k
Connections:
- removed net VBUS: C5.1, J3.7
- net 3.3V: now also C5.1
- net 5V: now also J4.2
- net B13: now also J4.6; no longer J3.3
- net B14: now also J4.7; no longer J3.2
- net B15: now also J4.8; no longer J3.1
- net B7: now also J4.3; no longer J3.6
- net B8: now also J4.4; no longer J3.5
- net B9: now also J4.5; no longer J3.4
- net D+: now also J6.D+; no longer X1G$1.3
- net D-: now also J6.D-; no longer X1G$1.2
- net GND: now also J4.1, J6.GND; no longer J3.8, U$6.3, X1G$1.5
- net ID: now also J6.ID; no longer X1G$1.4
- net VBUSUSB: now also J6.VBUS; no longer X1G$1.1
Other:
- moved on the sheet: C4, C5, D1, J1, J2, R2, R3, R4, U$2, U$3
